File: v1/arduino-theremin-v1.sch (KiCad schematic (older format))
At the start: 15 parts, among them P1 LV-EZ1 RANGEFINDER, SW1 SW_PUSH_B3F_1XXX, SW2 ON-OFF-ON SWITCH, U1 Arduino_Uno_R3_Shield

Commit message: v1.3, based on wickerlib, fixes the reversed rangefinder. Ordered from OSH Park.
Parts:
- removed LED1: ON, LEDs:LED-5MM, symbol Led_Small
- removed LED2: PLAYBACK, LEDs:LED-5MM, symbol Led_Small
- removed P1: LV-EZ1 RANGEFINDER, Wicker_Modules:LV_EZ1_Rangefinder, symbol CONN_01X07
- removed R1, R2: 220, Resistors_ThroughHole:Resistor_Horizontal_RM7mm, symbol R_Small
- removed RV1: POT, Wicker_Resistors_Pots:16mm_Rotary_Potentiometer, symbol POT
- removed SP1: SPEAKER, Pin_Headers:Pin_Header_Straight_1x02, symbol SPEAKER
- removed SW1: SW_PUSH_B3F_1XXX, Buttons_Switches_ThroughHole:SW_TH_Tactile_Omron_B3F-10xx, symbol SW_PUSH_B3F_1XXX
- removed SW2: ON-OFF-ON SWITCH, Wicker_Buttons_Switches:ESwitch_Series100_SPDT, symbol SWITCH_INV_MSM
- removed U1: Arduino_Uno_R3_Shield, Wicker_Shields:Arduino_Uno_R3_No_ICSP, symbol Arduino_Uno_R3_Shield
- added J1: LV-EZ1-RANGEFINDER, Wickerlib:LV_EZ1_Rangefinder, symbol LV-EZ1-RANGEFINDER
- added LED1: RECORD, Wickerlib:LED-5MM-2PIN, symbol LED-RED-2PIN-TH-MT4118-HR-A
- added LED2: PLAYBACK, Wickerlib:LED-5MM-2PIN, symbol LED-GREEN-2PIN-TH-MT2118-G-A
- added R1, R2: 220, Wickerlib:Resistor_Horizontal_RM7mm, symbol RES-220-5%-1/4W-TH-CFMINI
- added RV1: 10K, Wickerlib:P160-TRIMPOT, symbol TRIMPOT-10K-3PIN-TH-0.20W-P160KN
- added S1: 100SP3 ON-OFF-ON, Wickerlib:SW-100SP3, symbol SWITCH-TOGGLE-SPDT-5A-120V
- added SPK1: SPEAKER-8OHM-23MM-ROUND-2PIN, Wickerlib:Pin_Header_Straight_1x02, symbol SPEAKER-8OHM-23MM-ROUND-2PIN
- added SW1: B3F-1000, Wickerlib:SW-B3F-10XX, symbol SWITCH-TACT-SPDT-B3F-1000
- added U1: ARDUINO-UNO-SHIELD, Wickerlib:ARDU-UNOSHIELD, symbol ARDUINO-UNO-SHIELD
- CAP1, CAP2, CAP3: footprint Wicker_CapSense:CAPSENSE_CIRCLE_D10 -> Wickerlib:CAPSENSE-CIRCLE-D10
- R3, R4: footprint Resistors_ThroughHole:Resistor_Horizontal_RM7mm -> Wickerlib:Resistor_Horizontal_RM7mm; symbol R_Small -> RES-10K-5%-1/4W-TH-CFMINI
Connections:
- net labels added: A5_RECORD_LED
- net labels removed: A5_ON_LED
- wire segments 52 -> 50
- no-connect marks 23 -> 22
Other:
- note removed: "BW\n\nAN\nRX\nTX"
