File: hardware/arduino-theremin-v1.sch (KiCad schematic (older format))
At the start: 15 parts, among them J1 LV-EZ1-RANGEFINDER, SW1 B3F-1000, U1 ARDUINO-UNO-SHIELD

Commit message: Ported Arduino Theremin to use Wickerlib.
Parts:
- SPK1: value SPEAKER-8OHM-23MM-ROUND-2PIN -> 8 OHM; footprint Wickerlib:Pin_Header_Straight_1x02 -> Wickerlib:OSTVN02A150; Package UNDEFINED -> OSTVN02A150
Changed lines of the file:
@@
 $EndComp
 $Comp
-L +5V #PWR05
-U 1 1 572438D0
-P 8825 1575
-F 0 "#PWR05" H 8825 1425 50  0001 C CNN
-F 1 "+5V" H 8825 1715 50  0000 C CNN
-F 2 "" H 8825 1575 50  0000 C CNN
-F 3 "" H 8825 1575 50  0000 C CNN
-	1    8825 1575
-	-1   0    0    -1
-$EndComp
-$Comp
-L GND #PWR06
+L GND #PWR05
 U 1 1 57243924
 P 5800 2350
-F 0 "#PWR06" H 5800 2350 30  0001 C CNN
+F 0 "#PWR05" H 5800 2350 30  0001 C CNN
 F 1 "GND" H 5800 2280 30  0001 C CNN
 F 2 "" H 5800 2350 60  0000 C CNN
@@
 $EndComp
 $Comp
-L GND #PWR07
+L GND #PWR06
 U 1 1 57243EA6
 P 7225 2275
-F 0 "#PWR07" H 7225 2275 30  0001 C CNN
+F 0 "#PWR06" H 7225 2275 30  0001 C CNN
 F 1 "GND" H 7225 2205 30  0001 C CNN
 F 2 "" H 7225 2275 60  0000 C CNN
@@
 $EndComp
 $Comp
-L GND #PWR08
+L GND #PWR07
 U 1 1 57243EE7
 P 7625 2275
-F 0 "#PWR08" H 7625 2275 30  0001 C CNN
+F 0 "#PWR07" H 7625 2275 30  0001 C CNN
 F 1 "GND" H 7625 2205 30  0001 C CNN
 F 2 "" H 7625 2275 60  0000 C CNN
@@
 $EndComp
 $Comp
-L +5V #PWR09
+L +5V #PWR08
 U 1 1 5724467F
 P 8000 3650
-F 0 "#PWR09" H 8000 3500 50  0001 C CNN
+F 0 "#PWR08" H 8000 3500 50  0001 C CNN
 F 1 "+5V" H 8000 3790 50  0000 C CNN
 F 2 "" H 8000 3650 50  0000 C CNN
@@
 $EndComp
 $Comp
-L GND #PWR010
+L GND #PWR09
 U 1 1 572446E6
 P 8000 3925
-F 0 "#PWR010" H 8000 3925 30  0001 C CNN
+F 0 "#PWR09" H 8000 3925 30  0001 C CNN
 F 1 "GND" H 8000 3855 30  0001 C CNN
 F 2 "" H 8000 3925 60  0000 C CNN
@@
 $EndComp
 $Comp
-L GND #PWR011
+L GND #PWR010
 U 1 1 57244EF8
 P 8100 5050
-F 0 "#PWR011" H 8100 5050 30  0001 C CNN
+F 0 "#PWR010" H 8100 5050 30  0001 C CNN
 F 1 "GND" H 8100 4980 30  0001 C CNN
 F 2 "" H 8100 5050 60  0000 C CNN
@@
 $EndComp
 $Comp
-L GND #PWR012
+L GND #PWR011
 U 1 1 57244F39
 P 8500 5325
-F 0 "#PWR012" H 8500 5325 30  0001 C CNN
+F 0 "#PWR011" H 8500 5325 30  0001 C CNN
 F 1 "GND" H 8500 5255 30  0001 C CNN
 F 2 "" H 8500 5325 60  0000 C CNN
@@
 $EndComp
 $Comp
-L GND #PWR013
+L GND #PWR012
 U 1 1 57245851
 P 2825 4675
-F 0 "#PWR013" H 2825 4675 30  0001 C CNN
+F 0 "#PWR012" H 2825 4675 30  0001 C CNN
 F 1 "GND" H 2825 4605 30  0001 C CNN
 F 2 "" H 2825 4675 60  0000 C CNN
@@
 $EndComp
 $Comp
-L GND #PWR014
+L GND #PWR013
 U 1 1 57245E30
 P 3350 4675
-F 0 "#PWR014" H 3350 4675 30  0001 C CNN
+F 0 "#PWR013" H 3350 4675 30  0001 C CNN
 F 1 "GND" H 3350 4605 30  0001 C CNN
 F 2 "" H 3350 4675 60  0000 C CNN
@@
 $EndComp
 $Comp
-L SPEAKER-8OHM-23MM-ROUND-2PIN SPK1
-U 1 1 5724C38A
-P 8850 5000
-F 0 "SPK1" H 8850 5450 50  0000 L CNN
-F 1 "SPEAKER-8OHM-23MM-ROUND-2PIN" H 8850 5350 50  0000 L CNN
-F 2 "Wickerlib:Pin_Header_Straight_1x02" H 8850 4650 50  0001 C CIN
-F 3 "http://www.mallory-sonalert.com/specifications/PSR-23F08S-JQ.PDF" H 8850 5000 5   0001 C CNN
-F 4 "UNDEFINED" H 8850 4650 50  0001 C CIN "Package"
-F 5 "Mallory Sonalert" H 8850 4650 50  0001 C CIN "MF_Name"
-F 6 "PSR-23F08S-JQ" H 8850 4650 50  0001 C CIN "MF_PN"
-F 7 "Digikey" H 8850 4650 50  0001 C CIN "S1_Name"
-F 8 "458-1124-ND" H 8850 4650 50  0001 C CIN "S1_PN"
-F 9 "SPEAKER 8 OHM .25W 23MM ROUND" H 8850 4650 50  0001 C CIN "Description"
-F 10 "Not Verified" H 8850 4650 50  0001 C CIN "Verified"
-	1    8850 5000
-	1    0    0    -1
-$EndComp
-$Comp
 L TRIMPOT-10K-3PIN-TH-0.20W-P160KN RV1
 U 1 1 5724C6C3
@@
 	0    1    1    0
 $EndComp
+$Comp
+L SPEAKER-8OHM-23MM-ROUND-2PIN SPK1
+U 1 1 573835F3
+P 8850 5000
+F 0 "SPK1" H 8750 4800 50  0000 L CNN
+F 1 "8 OHM" H 8750 4725 50  0000 L CNN
+F 2 "Wickerlib:OSTVN02A150" H 8850 4650 50  0001 C CIN
+F 3 "http://www.mallory-sonalert.com/specifications/PSR-23F08S-JQ.PDF" H 8850 5000 5   0001 C CNN
+F 4 "OSTVN02A150" H 8850 4650 50  0001 C CIN "Package"
+F 5 "Mallory Sonalert" H 8850 4650 50  0001 C CIN "MF_Name"
+F 6 "PSR-23F08S-JQ" H 8850 4650 50  0001 C CIN "MF_PN"
+F 7 "Digikey" H 8850 4650 50  0001 C CIN "S1_Name"
+F 8 "458-1124-ND" H 8850 4650 50  0001 C CIN "S1_PN"
+F 9 "SPEAKER 8 OHM .25W 23MM ROUND" H 8850 4650 50  0001 C CIN "Description"
+F 10 "Not Verified" H 8850 4650 50  0001 C CIN "Verified"
+	1    8850 5000
+	1    0    0    -1
+$EndComp
+$Comp
+L +5V #PWR014
+U 1 1 573861A1
+P 8825 1575
+F 0 "#PWR014" H 8825 1425 50  0001 C CNN
+F 1 "+5V" H 8825 1715 50  0000 C CNN
+F 2 "" H 8825 1575 50  0000 C CNN
+F 3 "" H 8825 1575 50  0000 C CNN
+	1    8825 1575
+	1    0    0    -1
+$EndComp
 $EndSCHEMATC

Commit message: Added text on schematic to indicate A, C, F keys.
Other:
- note added: "A"
- note added: "C"
- note added: "F"
Changed lines of the file:
@@
 EESchema Schematic File Version 2
 LIBS:wickerlib
+LIBS:arduino-theremin-v1-cache
 EELAYER 25 0
 EELAYER END
@@
 	1    0    0    -1
 $EndComp
+Text Notes 5225 5225 0    79   ~ 0
+A
+Text Notes 6400 5700 0    79   ~ 0
+C
+Text Notes 6425 5225 0    79   ~ 0
+F
 $EndSCHEMATC

Commit message: Updated board file to match correct names for D8 and D9 PLAYBACK and RECORD. All done.
Connections:
- net D8_BTN_PLAYBACK renamed D8_BTN_RECORD
- net D9_BTN_RECORD renamed D9_BTN_PLAYBACK
Changed lines of the file:
@@
 D6_KEY2
 Text Label 5700 1750 0    60   ~ 0
-D9_BTN_RECORD
+D9_BTN_PLAYBACK
 Text Label 5700 1650 0    60   ~ 0
-D8_BTN_PLAYBACK
+D8_BTN_RECORD
 Text Label 5000 4175 0    60   ~ 0
 D5_KEY3
